File: micro_midi_w_fader/micro_midi_w_fader.kicad_pcb (KiCad board)
At the start: 2 copper layers, 222.3 x 173.2 mm, 94 parts, among them P1 Pad 1.7mm Hole 3.0mm, P2 Pad 1.7mm Hole 3.0mm, P3 Pad 1.7mm Hole 3.0mm, P4 Pad 1.7mm Hole 3.0mm, P5 Pad 1.7mm Hole 3.0mm, P6 Pad 1.7mm Hole 3.0mm, P7 Pad 1.7mm Hole 3.0mm, P8 Pad 1.7mm Hole 3.0mm

Commit message: cleaned repo and readme
Parts:
- C0, C1, C2, C3, GND1, L0, L1, L10, L11, L12, L13, L14, L15, L2, L3, L4, L5, L6, L7, L8, L9, R0, R1, R2, R3: footprint TestPoint:TestPoint_Plated_Hole_D3.0mm -> CustomLib:THROUGH HOLE PAD 1.7MM HOLE 3.0MM PAD
Routing:
- net Net-(D17-K): track 763.6 -> 755.2 mm
- net Net-(D31-A): track 131.6 -> 130.6 mm
Other:
- outline, holes or cut-outs redrawn

Commit message: reaaligned
Parts:
- moved F8 62.0 mm to (314.9, 114.0)
- moved S16 62.0 mm to (314.9, 215.4)
- moved S8 62.0 mm to (314.9, 191.6)
- moved D16 62.0 mm to (323.4, 219.3)
- moved D24 62.0 mm to (313.6, 196.7)
- moved D32 62.0 mm to (313.6, 220.5)
- moved D8 62.0 mm to (323.4, 195.5)
- moved F6 61.8 mm to (257.9, 114.0)
- moved D14 61.7 mm to (267.4, 219.3)
- moved D22 61.7 mm to (256.6, 196.7)
- moved D30 61.7 mm to (256.6, 220.5)
- moved D6 61.7 mm to (267.4, 195.5)
- moved S14 61.7 mm to (257.9, 215.4)
- moved S6 61.7 mm to (257.9, 191.6)
- moved F2 61.6 mm to (143.9, 114.0)
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Routing:
- net Net-(D21-A): track 82.1 -> 79.4 mm
- net Net-(D17-K): track 755.2 -> 752.7 mm
- net Net-(D17-A): track 68.7 -> 66.9 mm
- net Net-(D5-K): track 293.4 -> 291.7 mm
- net Net-(D24-A): track 147.7 -> 146.2 mm
- net Net-(D13-K): track 311.9 -> 310.3 mm
- net Net-(D32-A): track 154.5 -> 153.0 mm
- net Net-(D30-A): track 99.4 -> 98.2 mm
- net Net-(D22-A): track 97.6 -> 96.5 mm
- net Net-(D23-A): track 127.1 -> 125.9 mm
- net Net-(D27-A): track 64.1 -> 63.0 mm
- net Net-(C0-Pad1): track 201.2 -> 200.1 mm
- net Net-(C3-Pad1): track 241.5 -> 240.5 mm
- net Net-(D31-A): track 130.6 -> 129.7 mm
- net Net-(D28-A): track 52.6 -> 51.6 mm
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Other:
- board size 222.3 x 173.2 mm -> 222.2 x 173.2 mm
